File: ArduinoMegaShield.kicad_pcb (KiCad board)
At the start: 2 copper layers, 101.6 x 53.3 mm, 13 parts, among them J1 Power, J2 PWM, J3 Analog, J4 PWM, J5 Analog, J6 Communication, J7 Digital

Commit message: Finished Schematic
Parts:
- added C1: 100uF, Capacitor_THT:CP_Radial_D6.3mm_P2.50mm, F.Cu at (75.1, 75.5)
- added C2: 100uF, Capacitor_THT:CP_Radial_D6.3mm_P2.50mm, F.Cu at (75.1, 83.3)
- added J10: Conn_01x04_Socket, Connector_PinSocket_2.54mm:PinSocket_1x04_P2.54mm_Vertical, F.Cu at (219.7, 69.1)
- added J11: Conn_01x02_Socket, Connector_PinSocket_2.54mm:PinSocket_1x02_P2.54mm_Vertical, F.Cu at (42.8, 104.8)
- added J12: Conn_01x02_Socket, Connector_PinSocket_2.54mm:PinSocket_1x02_P2.54mm_Vertical, F.Cu at (47.4, 104.8)
- added J13: Conn_01x02_Socket, Connector_PinSocket_2.54mm:PinSocket_1x02_P2.54mm_Vertical, F.Cu at (52.0, 104.8)
- added J14: Conn_01x02_Socket, Connector_PinSocket_2.54mm:PinSocket_1x02_P2.54mm_Vertical, F.Cu at (56.6, 104.8)
- added J15: Conn_01x04, Connector_JST:JST_EH_S4B-EH_1x04_P2.50mm_Horizontal, F.Cu at (139.3, 113.9)
- added J16: Conn_01x04, Connector_JST:JST_EH_S4B-EH_1x04_P2.50mm_Horizontal, F.Cu at (154.6, 113.9)
- added J17: Conn_01x10_Socket, Connector_PinSocket_2.54mm:PinSocket_1x10_P2.54mm_Vertical, F.Cu at (211.2, 62.1)
- added J18: Barrel_Jack_Switch, Connector_BarrelJack:BarrelJack_CUI_PJ-102AH_Horizontal, F.Cu at (106.8, 71.6)
- added J8: Conn_01x04_Socket, Connector_PinSocket_2.54mm:PinSocket_1x04_P2.54mm_Vertical, F.Cu at (212.1, 42.7)
- added J9: Conn_01x04_Socket, Connector_PinSocket_2.54mm:PinSocket_1x04_P2.54mm_Vertical, F.Cu at (216.7, 42.7)
- added Q1: IRLB8721PBF, Package_TO_SOT_THT:TO-220-3_Vertical, F.Cu at (47.5, 54.2)
- added Q2: IRLB8721PBF, Package_TO_SOT_THT:TO-220-3_Vertical, F.Cu at (47.5, 60.1)
- added Q3: IRLB8721PBF, Package_TO_SOT_THT:TO-220-3_Vertical, F.Cu at (47.5, 66.1)
- added Q4: IRLB8721PBF, Package_TO_SOT_THT:TO-220-3_Vertical, F.Cu at (47.5, 72.0)
- added Q5: IRLB8721PBF, Package_TO_SOT_THT:TO-220-3_Vertical, F.Cu at (47.5, 78.0)
- added Q6: IRLB8721PBF, Package_TO_SOT_THT:TO-220-3_Vertical, F.Cu at (47.5, 84.0)
- added Q7: IRLB8721PBF, Package_TO_SOT_THT:TO-220-3_Vertical, F.Cu at (47.5, 89.9)
- added R1: 10K, Resistor_SMD:R_0805_2012Metric_Pad1.20x1.40mm_HandSolder, F.Cu at (58.1, 51.7)
- added R2: 10K, Resistor_SMD:R_0805_2012Metric_Pad1.20x1.40mm_HandSolder, F.Cu at (58.1, 54.7)
- added R3: 10K, Resistor_SMD:R_0805_2012Metric_Pad1.20x1.40mm_HandSolder, F.Cu at (82.6, 73.0)
- added R4: 10K, Resistor_SMD:R_0805_2012Metric_Pad1.20x1.40mm_HandSolder, F.Cu at (82.6, 76.0)
- added R5: 10K, Resistor_SMD:R_0805_2012Metric_Pad1.20x1.40mm_HandSolder, F.Cu at (82.6, 78.9)
- added R6: 10K, Resistor_SMD:R_0805_2012Metric_Pad1.20x1.40mm_HandSolder, F.Cu at (82.6, 81.8)
- added R7: 10K, Resistor_SMD:R_0805_2012Metric_Pad1.20x1.40mm_HandSolder, F.Cu at (82.6, 84.8)
- added U1: MP6500_Pololu, Module:Pololu_Breakout-16_15.2x20.3mm, F.Cu at (79.0, 106.9)
- added U2: MP6500_Pololu, Module:Pololu_Breakout-16_15.2x20.3mm, F.Cu at (120.8, 63.6)
- renumbered J3 to J2, J5 to J3, J7 to J4, J2 to J5, J4 to J6, J6 to J7
