File: _autosave-ArduinoMegaShield.kicad_pcb (KiCad board)
At the start: 2 copper layers, 101.6 x 53.3 mm, 42 parts, among them J1 Power, J10 Conn_01x04_Socket, J11 Conn_01x02_Socket, J12 Conn_01x02_Socket, J13 Conn_01x02_Socket, J14 Conn_01x02_Socket, J15 Conn_01x04, J16 Conn_01x04, J17 Conn_01x10_Socket, J18 Barrel_Jack_Switch, J2 Analog, J3 Analog, J4 Digital, J5 PWM, J6 PWM, J7 Communication, J8 Conn_01x04_Socket, J9 Conn_01x04_Socket, Q1 IRLB8721PBF, Q2 IRLB8721PBF, Q3 IRLB8721PBF, Q4 IRLB8721PBF, Q5 IRLB8721PBF, Q6 IRLB8721PBF, Q7 IRLB8721PBF, U1 MP6500_Pololu, U2 MP6500_Pololu

Commit message: Update
Parts:
- J15, J16: footprint Connector_JST:JST_EH_S4B-EH_1x04_P2.50mm_Horizontal -> Connector_JST:JST_XH_B4B-XH-A_1x04_P2.50mm_Vertical
- moved J13 28.4 mm to (77.5, 117.2)
- moved J11 28.4 mm to (68.3, 117.2)
- moved J12 28.4 mm to (72.9, 117.2)
- moved J14 28.4 mm to (82.1, 117.2)
- moved J17 27.8 mm to (210.2, 89.9)
- moved J9 11.6 mm to (218.8, 54.1), turned to -90 degrees
- moved J8 9.58 mm to (218.8, 49.5), turned to -90 degrees
- moved J10 8.87 mm to (211.8, 65.1), turned to 90 degrees
- moved J18 5.87 mm to (110.2, 76.3), turned to -90 degrees
- moved J16 5.21 mm to (171.1, 133.6)
- moved U2 5.07 mm to (179.9, 114.7)
- moved C1 4.76 mm to (179.1, 132.8)
- moved C2 2.65 mm to (143.7, 132.1)
- moved J15 2.02 mm to (135.7, 132.7)
- moved U1 2.02 mm to (144.4, 114.0)
